File: schematic/eprom_prog.sch (EAGLE design)
At the start: 50 parts, among them IC1 MC33063/MC34063P, K1 G5V1, K2 G5V1, K3 G5V1, K4 G5V1, K5 G5V1, K6 G5V1, Q1 BS170, Q2 BS170, Q3 BS170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

Commit message: schematic: BOM and pdf export
Other:
- note added: "V1.0"
Changed lines of the file:
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@@
 <plain>
 <text x="289.56" y="25.4" size="5.08" layer="91">CPU &amp; Sockel</text>
+<text x="375.92" y="7.62" size="2.54" layer="91">V1.0</text>
 </plain>
 <instances>
@@
 <plain>
 <text x="289.56" y="25.4" size="5.08" layer="91">VPP Supply</text>
+<text x="375.92" y="7.62" size="2.54" layer="91">V1.0</text>
 </plain>
 <instances>
